Commit message: Added realsense to gazebo and its working

File: mycobot_280pi_gazebo/urdf/mycobot_280pi_gazebo.xacro (robot description, xacro)
@@ -1,4 +1,12 @@
 <?xml version="1.0" ?>
 <robot xmlns:xacro="http://wiki.ros.org/xacro" name="mycobot_280pi">
+  <xacro:property name="M_PI" value="3.1415926535897931" />
+  <xacro:property name="d435_cam_width" value="0.090"/>
+  <xacro:property name="d435_cam_height" value="0.025"/>
+  <xacro:property name="d435_cam_depth" value="0.02505"/>
+  <xacro:property name="d435_cam_depth_to_infra1_offset" value="0.0"/>
+  <xacro:property name="d435_cam_depth_to_infra2_offset" value="-0.050"/>
+  <xacro:property name="d435_cam_depth_to_color_offset" value="0.015"/>
+  <xacro:property name="camera_tilt_angle_deg" value="45"/>
     <gazebo>
         <plugin filename="gz_ros2_control-system" name="gz_ros2_control::GazeboSimROS2ControlPlugin">
@@ -9,3 +17,142 @@
         </plugin>
     </gazebo>
+<!--                   -->
+  <link name="torso_link">
+    <inertial>
+      <origin xyz="0 0 0.50" />
+      <mass value="2.5" />
+      <inertia ixx="0.8" ixy="0.0" ixz="0.0" iyy="0.8" iyz="0.0" izz="0.8" />
+    </inertial>
+    <visual name="holder">
+      <origin xyz="0 0 0.25" rpy="0 0 0" />
+      <material name="LightGrey">
+        <color rgba="0.7 0.7 0.7 1.0"/>
+      </material>
+      <geometry>
+        <cylinder radius="0.005" length="0.5"/>
+      </geometry>
+    </visual>
+    <visual name="base">
+      <origin xyz="0 0 0" rpy="0 0 0" />
+      <material name="LightGrey">
+        <color rgba="0.7 0.7 0.7 1.0"/>
+      </material>
+      <geometry>
+        <box size="0.15 0.10 0.06" />
+      </geometry>
+    </visual>
+    <collision name="holder">
+      <origin xyz="0 0 0.25" rpy="0 0 0" />
+      <geometry>
+        <cylinder radius="0.005" length="0.6"/>
+      </geometry>
+    </collision>
+    <collision name="base">
+      <origin xyz="0 0 0.0" rpy="0 0 0" />
+      <geometry>
+        <box size="0.15 0.10 0.06" />
+      </geometry>
+    </collision>
+  </link>
+  <joint name="base_link_to_torso_link" type="fixed">
+    <parent link="g_base"/>
+    <child link="torso_link"/>
+    <origin xyz="0.8 0 0" rpy="0 0 1.57"/>
+  </joint>
+  <joint name="camera_head_joint" type="fixed">
+    <parent link="torso_link"/>
+    <child link="camera_head_link" />
+    <origin xyz="0 0.01 0.50" rpy="0.0 ${camera_tilt_angle_deg * M_PI / 180} ${M_PI/2}"/>
+  </joint>
+  <link name="camera_head_link">
+    <visual>
+      <origin xyz="0 0 0" rpy="${M_PI/2} 0.0 ${M_PI/2}"/>
+      <geometry>
+        <mesh filename="file://$(find mycobot_280pi_description)/meshes/d435.stl" />
+      </geometry>
+      <material name="aluminum">
+        <color rgba="0.5 0.5 0.5 1"/>
+      </material>
+    </visual>
+    <collision>
+      <origin xyz="0 0 0" rpy="0 0 0"/>
+      <geometry>
+        <box size="${d435_cam_depth} ${d435_cam_width} ${d435_cam_height}"/>
+      </geometry>
+    </collision>
+    <inertial>
+      <mass value="0.072" />
+      <origin xyz="0 0 0" />
+      <inertia ixx="0.003881243" ixy="0.0" ixz="0.0" iyy="0.000498940" iyz="0.0" izz="0.003879257" />
+    </inertial>
+  </link>
+  <joint name="camera_head_depth_joint" type="fixed">
+    <origin xyz="0 0 0" rpy="0 0 0"/>
+    <parent link="camera_head_link"/>
+    <child link="camera_head_depth_frame" />
+  </joint>
+  <link name="camera_head_depth_frame"/>
+  <joint name="camera_head_depth_optical_joint" type="fixed">
+    <origin xyz="0 0 0" rpy="${-M_PI/2} 0 ${-M_PI/2}" />
+    <parent link="camera_head_depth_frame" />
+    <child link="camera_head_depth_optical_frame" />
+  </joint>
+  <link name="camera_head_depth_optical_frame"/>
+  <joint name="camera_head_infra1_joint" type="fixed">
+    <origin xyz="0 ${d435_cam_depth_to_infra1_offset} 0" rpy="0 0 0" />
+    <parent link="camera_head_link" />
+    <child link="camera_head_infra1_frame" />
+  </joint>
+  <link name="camera_head_infra1_frame"/>
+  <joint name="camera_head_infra1_optical_joint" type="fixed">
+    <origin xyz="0 0 0" rpy="${-M_PI/2} 0 ${-M_PI/2}" />
+    <parent link="camera_head_infra1_frame" />
+    <child link="camera_head_infra1_optical_frame" />
+  </joint>
+  <link name="camera_head_infra1_optical_frame"/>
+  <joint name="camera_head_infra2_joint" type="fixed">
+    <origin xyz="0 ${d435_cam_depth_to_infra2_offset} 0" rpy="0 0 0" />
+    <parent link="camera_head_link" />
+    <child link="camera_head_infra2_frame" />
+  </joint>
+  <link name="camera_head_infra2_frame"/>
+  <joint name="camera_head_infra2_optical_joint" type="fixed">
+    <origin xyz="0 0 0" rpy="${-M_PI/2} 0 ${-M_PI/2}" />
+    <parent link="camera_head_infra2_frame" />
+    <child link="camera_head_infra2_optical_frame" />
+  </joint>
+  <link name="camera_head_infra2_optical_frame"/>
+  <joint name="camera_head_color_joint" type="fixed">
+    <origin xyz="0 ${d435_cam_depth_to_color_offset} 0" rpy="0 0 0" />
+    <parent link="camera_head_link" />
+    <child link="camera_head_color_frame" />
+  </joint>
+  <link name="camera_head_color_frame"/>
+  <joint name="camera_head_color_optical_joint" type="fixed">
+    <origin xyz="0 0 0" rpy="${-M_PI/2} 0 ${-M_PI/2}" />
+    <parent link="camera_head_color_frame" />
+    <child link="camera_head_color_optical_frame" />
+  </joint>
+  <link name="camera_head_color_optical_frame"/>
+  <gazebo reference="camera_head_link">
+    <sensor name="camera_head" type="rgbd_camera">
+      <camera>
+        <horizontal_fov>1.5184</horizontal_fov>
+        <image>
+          <width>424</width>
+          <height>240</height>
+        </image>
+        <clip>
+          <near>0.05</near>
+          <far>1.5</far>
+        </clip>
+        <optical_frame_id>camera_head_depth_optical_frame</optical_frame_id>
+      </camera>
+      <always_on>1</always_on>
+      <gz_frame_id>camera_head_link</gz_frame_id>
+      <topic>camera_head</topic>
+      <update_rate>5</update_rate>
+      <visualize>true</visualize>
+    </sensor>
+  </gazebo>
 </robot>

Commit message: Added realsense parameters and position

File: mycobot_280pi_gazebo/urdf/mycobot_280pi_gazebo.xacro (robot description, xacro)
@@ -8,5 +8,5 @@
   <xacro:property name="d435_cam_depth_to_infra2_offset" value="-0.050"/>
   <xacro:property name="d435_cam_depth_to_color_offset" value="0.015"/>
-  <xacro:property name="camera_tilt_angle_deg" value="45"/>
+  <xacro:property name="camera_tilt_angle_deg" value="5"/>
     <gazebo>
         <plugin filename="gz_ros2_control-system" name="gz_ros2_control::GazeboSimROS2ControlPlugin">
@@ -58,10 +58,11 @@
     <parent link="g_base"/>
     <child link="torso_link"/>
-    <origin xyz="0.8 0 0" rpy="0 0 1.57"/>
+    <origin xyz="0.7 0 0" rpy="0 0 1.57"/>
+<!--   <origin xyz="0.8 0 0" rpy="0 0 1.57"/>  -->
   </joint>
   <joint name="camera_head_joint" type="fixed">
     <parent link="torso_link"/>
     <child link="camera_head_link" />
-    <origin xyz="0 0.01 0.50" rpy="0.0 ${camera_tilt_angle_deg * M_PI / 180} ${M_PI/2}"/>
+   <origin xyz="0 0.01 0.20" rpy="0.0 ${camera_tilt_angle_deg * M_PI / 180} ${M_PI/2}"/>
   </joint>
   <link name="camera_head_link">
@@ -140,6 +141,6 @@
         <horizontal_fov>1.5184</horizontal_fov>
         <image>
-          <width>424</width>
-          <height>240</height>
+          <width>640</width>
+          <height>480</height>
         </image>
         <clip>
