Commit message: Added sim and real vision node setup

File: mycobot_280pi_gazebo/urdf/mycobot_280pi_gazebo_real.xacro (robot description, xacro)
@@ -9,4 +9,6 @@
   <xacro:property name="d435_cam_depth_to_color_offset" value="0.015"/>
   <xacro:property name="camera_tilt_angle_deg" value="5"/>
+  <xacro:property name="distance_of_cam" value="0.7"/>
+  <xacro:property name="height_of_cam" value="0.2"/>
     <gazebo>
         <plugin filename="gz_ros2_control-system" name="gz_ros2_control::GazeboSimROS2ControlPlugin">
@@ -58,5 +60,5 @@
     <parent link="g_base"/>
     <child link="torso_link"/>
-    <origin xyz="0.7 0 0" rpy="0 0 1.57"/>
+    <origin xyz="${distance_of_cam} 0 0" rpy="0 0 1.57"/>
 <!--   <origin xyz="0.8 0 0" rpy="0 0 1.57"/>  -->
   </joint>
@@ -64,5 +66,5 @@
     <parent link="torso_link"/>
     <child link="camera_link" />
-   <origin xyz="0 0.01 0.20" rpy="0.0 ${camera_tilt_angle_deg * M_PI / 180} ${M_PI/2}"/>
+   <origin xyz="0 0.01 ${height_of_cam}" rpy="0.0 ${camera_tilt_angle_deg * M_PI / 180} ${M_PI/2}"/>
   </joint>
   <link name="camera_link">
