Commit message: Updated gripper and tested working

File: mycobot_280pi_description/urdf/mycobot_280_pi.urdf (robot description, URDF)
Before this commit: robot firefighter, 8 links, 7 joints
Links:
- added link gripper_base, mass 0.07; collision box size=0.065 0.025 0.025; visual mesh filename=package://mycobot_280pi_description/meshes/gripper_base.dae
- added link gripper_left1, mass 0.007; collision box size=0.013 0.02 0.015; visual mesh filename=package://mycobot_280pi_description/meshes/gripper_left1.dae
- added link gripper_left2, mass 0.007; collision box size=0.02 0.02 0.02; visual mesh filename=package://mycobot_280pi_description/meshes/gripper_left2.dae
- added link gripper_left3, mass 0.007; collision box size=0.01 0.01 0.01; visual mesh filename=package://mycobot_280pi_description/meshes/gripper_left3.dae
- added link gripper_right1, mass 0.007; collision box size=0.013 0.02 0.015; visual mesh filename=package://mycobot_280pi_description/meshes/gripper_right1.d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
- added link gripper_right2, mass 0.007; collision box size=0.02 0.02 0.02; visual mesh filename=package://mycobot_280pi_description/meshes/gripper_right2.d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
- added link gripper_right3, mass 0.007; collision box size=0.01 0.01 0.01; visual mesh filename=package://mycobot_280pi_description/meshes/gripper_right3.d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
Joints:
- added joint gripper_base_to_gripper_left2: type revolute, parent gripper_base, child gripper_left2, origin xyz=-0.005 0.027 0 rpy=0 0 0, axis 0 0 1, limit lower=-0.8 upper=0.5 effort=1000 velocity=0, mimic joint=gripper_controller multiplier=1.0 offset=0
- added joint gripper_base_to_gripper_right2: type revolute, parent gripper_base, child gripper_right2, origin xyz=0.005 0.027 0 rpy=0 0 0, axis 0 0 1, limit lower=-0.5 upper=0.8 effort=1000 velocity=0, mimic joint=gripper_controller multiplier=-1.0 offset=0
- added joint gripper_base_to_gripper_right3: type revolute, parent gripper_base, child gripper_right3, origin xyz=0.012 0.005 0 rpy=0 0 0, axis 0 0 1, limit lower=-0.15 upper=0.7 effort=1000 velocity=0, mimic joint=gripper_controller multiplier=-1.0 offset=0
- added joint gripper_controller: type revolute, parent gripper_base, child gripper_left3, origin xyz=-0.012 0.005 0 rpy=0 0 0, axis 0 0 1, limit lower=-0.8 upper=0.15 effort=1000 velocity=0
- added joint gripper_left3_to_gripper_left1: type revolute, parent gripper_left3, child gripper_left1, origin xyz=-0.027 0.016 0 rpy=0 0 0, axis 0 0 1, limit lower=-0.5 upper=0.5 effort=1000 velocity=0, mimic joint=gripper_controller multiplier=-1.0 offset=0
- added joint gripper_right3_to_gripper_right1: type revolute, parent gripper_right3, child gripper_right1, origin xyz=0.027 0.016 0 rpy=0 0 0, axis 0 0 1, limit lower=-0.5 upper=0.5 effort=1000 velocity=0, mimic joint=gripper_controller multiplier=1.0 offset=0
- added joint joint6flange_to_gripper_base: type fixed, parent joint6_flange, child gripper_base, origin xyz=0 0 0.034 rpy=1.579 0 0

Commit message: Added inertial values

File: mycobot_280pi_description/urdf/mycobot_280_pi.urdf (robot description, URDF)
Before this commit: robot firefighter, 15 links, 14 joints
Links:
- link g_base: mass None -> 0.33
- link joint1: mass None -> 0.12
- link joint2: mass None -> 0.19
- link joint3: mass None -> 0.16
- link joint4: mass None -> 0.124
- link joint5: mass None -> 0.11
- link joint6: mass None -> 0.0739
- link joint6_flange: mass None -> 0.035

Commit message: mycobot controller is working, need to fix link

File: mycobot_280pi_description/urdf/mycobot_280_pi.urdf (robot description, URDF)
Before this commit: robot mycobot_280pi, 15 links, 14 joints
Links:
- link g_base: geometry collision mesh filename=file://$(find mycobot_280pi_description)/meshes/G_base.dae; visual mesh filename=file://$(find mycobot_280pi_description)/meshes/G_base.dae
- link gripper_base: geometry collision box size=0.065 0.025 0.025; visual mesh filename=file://$(find mycobot_280pi_description)/meshes/gripper_bas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
- link gripper_left1: geometry collision box size=0.013 0.02 0.015; visual mesh filename=file://$(find mycobot_280pi_description)/meshes/gripper_lef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
- link gripper_left2: geometry collision box size=0.02 0.02 0.02; visual mesh filename=file://$(find mycobot_280pi_description)/meshes/gripper_lef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
- link gripper_left3: geometry collision box size=0.01 0.01 0.01; visual mesh filename=file://$(find mycobot_280pi_description)/meshes/gripper_lef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
- link gripper_right1: geometry collision box size=0.013 0.02 0.015; visual mesh filename=file://$(find mycobot_280pi_description)/meshes/gripper_rig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
- link gripper_right2: geometry collision box size=0.02 0.02 0.02; visual mesh filename=file://$(find mycobot_280pi_description)/meshes/gripper_rig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
- link gripper_right3: geometry collision box size=0.01 0.01 0.01; visual mesh filename=file://$(find mycobot_280pi_description)/meshes/gripper_rig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
- link joint1: geometry collision mesh filename=file://$(find mycobot_280pi_description)/meshes/link1.dae; visual mesh filename=file://$(find mycobot_280pi_description)/meshes/link1.dae
- link joint2: geometry collision mesh filename=file://$(find mycobot_280pi_description)/meshes/link2.dae; visual mesh filename=file://$(find mycobot_280pi_description)/meshes/link2.dae
- link joint3: geometry collision mesh filename=file://$(find mycobot_280pi_description)/meshes/link3.dae; visual mesh filename=file://$(find mycobot_280pi_description)/meshes/link3.dae
- link joint4: geometry collision mesh filename=file://$(find mycobot_280pi_description)/meshes/link4.dae; visual mesh filename=file://$(find mycobot_280pi_description)/meshes/link4.dae
- link joint5: geometry collision mesh filename=file://$(find mycobot_280pi_description)/meshes/link5.dae; visual mesh filename=file://$(find mycobot_280pi_description)/meshes/link5.dae
- link joint6: geometry collision mesh filename=file://$(find mycobot_280pi_description)/meshes/link6.dae; visual mesh filename=file://$(find mycobot_280pi_description)/meshes/link6.dae
- link joint6_flange: geometry collision mesh filename=file://$(find mycobot_280pi_description)/meshes/link7.dae; visual mesh filename=file://$(find mycobot_280pi_description)/meshes/link7.dae

Commit message: Fixed gazebo joint issues, its loading properly

File: mycobot_280pi_description/urdf/mycobot_280_pi.urdf (robot description, URDF)
Before this commit: robot mycobot_280pi, 15 links, 14 joints
Joints:
- joint joint2_to_joint1: limit lower=-3.14 upper=3.14159 effort=1000.0 velocity=0 -> lower=-3.14 upper=3.14159 effort=56.0 velocity=2.79
- joint joint3_to_joint2: limit lower=-3.14 upper=3.14159 effort=1000.0 velocity=0 -> lower=-3.14 upper=3.14159 effort=56.0 velocity=2.79
- joint joint4_to_joint3: limit lower=-3.14 upper=3.14159 effort=1000.0 velocity=0 -> lower=-3.14 upper=3.14159 effort=56.0 velocity=2.79
- joint joint5_to_joint4: limit lower=-3.14 upper=3.14159 effort=1000.0 velocity=0 -> lower=-3.14 upper=3.14159 effort=56.0 velocity=2.79
- joint joint6_to_joint5: limit lower=-3.14 upper=3.14159 effort=1000.0 velocity=0 -> lower=-3.14 upper=3.14159 effort=56.0 velocity=2.79
- joint joint6output_to_joint6: limit lower=-3.14 upper=3.14159 effort=1000.0 velocity=0 -> lower=-3.14 upper=3.14159 effort=56.0 velocity=2.79

Commit message: Updated docker file to include rqt plugins

File: mycobot_280pi_description/urdf/mycobot_280_pi.urdf (robot description, URDF)
Before this commit: robot mycobot_280pi, 15 links, 14 joints
Links:
- link gripper_base: geometry collision box size=0.01 0.01 0.01; visual mesh filename=file://$(find mycobot_280pi_description)/meshes/gripper_bas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
- link gripper_left1: geometry collision box size=0.01 0.01 0.01; visual mesh filename=file://$(find mycobot_280pi_description)/meshes/gripper_lef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
- link gripper_left2: geometry collision box size=0.01 0.01 0.01; visual mesh filename=file://$(find mycobot_280pi_description)/meshes/gripper_lef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
- link gripper_right1: geometry collision box size=0.01 0.01 0.01; visual mesh filename=file://$(find mycobot_280pi_description)/meshes/gripper_rig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
- link gripper_right2: geometry collision box size=0.01 0.01 0.01; visual mesh filename=file://$(find mycobot_280pi_description)/meshes/gripper_rig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

Commit message: Updated URDF again from description package and planning to add inertia again, moveit config and description are ready

File: mycobot_280pi_description/urdf/mycobot_280_pi.urdf (robot description, URDF)
Before this commit: robot mycobot_280pi, 15 links, 14 joints
Links:
- link g_base: mass 0.33 -> None; geometry collision mesh filename=package://mycobot_description/urdf/mycobot_280_pi/G_base.dae; visual mesh filename=package://mycobot_description/urdf/mycobot_280_pi/G_base.dae
- link joint1: mass 0.12 -> None; geometry collision mesh filename=package://mycobot_description/urdf/mycobot_280_pi/joint1_pi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; visual mesh filename=package://mycobot_description/urdf/mycobot_280_pi/joint1_pi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
- link joint2: mass 0.19 -> None; geometry collision mesh filename=package://mycobot_description/urdf/mycobot_280_pi/joint2.dae; visual mesh filename=package://mycobot_description/urdf/mycobot_280_pi/joint2.dae
- link joint3: mass 0.16 -> None; geometry collision mesh filename=package://mycobot_description/urdf/mycobot_280_pi/joint3.dae; visual mesh filename=package://mycobot_description/urdf/mycobot_280_pi/joint3.dae
- link joint4: mass 0.124 -> None; geometry collision mesh filename=package://mycobot_description/urdf/mycobot_280_pi/joint4.dae; visual mesh filename=package://mycobot_description/urdf/mycobot_280_pi/joint4.dae
- link joint5: mass 0.11 -> None; geometry collision mesh filename=package://mycobot_description/urdf/mycobot_280_pi/joint5.dae; visual mesh filename=package://mycobot_description/urdf/mycobot_280_pi/joint5.dae
- link joint6: mass 0.0739 -> None; geometry collision mesh filename=package://mycobot_description/urdf/mycobot_280_pi/joint6.dae; visual mesh filename=package://mycobot_description/urdf/mycobot_280_pi/joint6.dae
- link joint6_flange: mass 0.035 -> None; geometry collision mesh filename=package://mycobot_description/urdf/mycobot_280_pi/joint7.dae; visual mesh filename=package://mycobot_description/urdf/mycobot_280_pi/joint7.dae
Joints:
- joint joint2_to_joint1: limit lower=-3.14 upper=3.14159 effort=56.0 velocity=2.79 -> lower=-3.14 upper=3.14159 effort=1000.0 velocity=0
- joint joint3_to_joint2: limit lower=-3.14 upper=3.14159 effort=56.0 velocity=2.79 -> lower=-3.14 upper=3.14159 effort=1000.0 velocity=0
- joint joint4_to_joint3: limit lower=-3.14 upper=3.14159 effort=56.0 velocity=2.79 -> lower=-3.14 upper=3.14159 effort=1000.0 velocity=0
- joint joint5_to_joint4: limit lower=-3.14 upper=3.14159 effort=56.0 velocity=2.79 -> lower=-3.14 upper=3.14159 effort=1000.0 velocity=0
- joint joint6_to_joint5: limit lower=-3.14 upper=3.14159 effort=56.0 velocity=2.79 -> lower=-3.14 upper=3.14159 effort=1000.0 velocity=0
- joint joint6output_to_joint6: limit lower=-3.14 upper=3.14159 effort=56.0 velocity=2.79 -> lower=-3.14 upper=3.14159 effort=1000.0 velocity=0

Commit message: Gazebo with new model working, need to tune controller parameter

File: mycobot_280pi_description/urdf/mycobot_280_pi.urdf (robot description, URDF)
Before this commit: robot mycobot_280pi, 15 links, 14 joints
Links:
- link g_base: mass None -> 0.33; geometry collision mesh filename=file://$(find mycobot_280pi_description)/meshes/G_base.dae; visual mesh filename=file://$(find mycobot_280pi_description)/meshes/G_base.dae
- link joint1: mass None -> 0.12; geometry collision mesh filename=file://$(find mycobot_280pi_description)/meshes/joint1_pi.d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 scale=0.001 0.001 0.001; visual mesh filename=file://$(find mycobot_280pi_description)/meshes/joint1_pi.d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 scale=0.001 0.001 0.001
- link joint2: mass None -> 0.19; geometry collision mesh filename=file://$(find mycobot_280pi_description)/meshes/joint2.dae; visual mesh filename=file://$(find mycobot_280pi_description)/meshes/joint2.dae
- link joint3: mass None -> 0.16; geometry collision mesh filename=file://$(find mycobot_280pi_description)/meshes/joint3.dae; visual mesh filename=file://$(find mycobot_280pi_description)/meshes/joint3.dae
- link joint4: mass None -> 0.124; geometry collision mesh filename=file://$(find mycobot_280pi_description)/meshes/joint4.dae; visual mesh filename=file://$(find mycobot_280pi_description)/meshes/joint4.dae
- link joint5: mass None -> 0.11; geometry collision mesh filename=file://$(find mycobot_280pi_description)/meshes/joint5.dae scale=0.001 0.001 0.001; visual mesh filename=file://$(find mycobot_280pi_description)/meshes/joint5.dae scale=0.001 0.001 0.001
- link joint6: mass None -> 0.0739; geometry collision mesh filename=file://$(find mycobot_280pi_description)/meshes/joint6.dae; visual mesh filename=file://$(find mycobot_280pi_description)/meshes/joint6.dae
- link joint6_flange: mass None -> 0.035; geometry collision mesh filename=file://$(find mycobot_280pi_description)/meshes/joint7.dae; visual mesh filename=file://$(find mycobot_280pi_description)/meshes/joint7.dae

Commit message: Gazebo model and pi model is working good, now checking gripper

File: mycobot_280pi_description/urdf/mycobot_280_pi.urdf (robot description, URDF)
Before this commit: robot mycobot_280pi, 15 links, 14 joints
Joints:
- joint gripper_base_to_gripper_left2: limit lower=-0.8 upper=0.5 effort=1000 velocity=0 -> lower=-0.8 upper=0.5 effort=${effort} velocity=${velocity}
- joint gripper_base_to_gripper_right2: limit lower=-0.5 upper=0.8 effort=1000 velocity=0 -> lower=-0.5 upper=0.8 effort=${effort} velocity=${velocity}
- joint gripper_base_to_gripper_right3: limit lower=-0.15 upper=0.7 effort=1000 velocity=0 -> lower=-0.15 upper=0.7 effort=${effort} velocity=${velocity}
- joint gripper_controller: limit lower=-0.8 upper=0.15 effort=1000 velocity=0 -> lower=-0.8 upper=0.15 effort=${effort} velocity=${velocity}
- joint gripper_left3_to_gripper_left1: limit lower=-0.5 upper=0.5 effort=1000 velocity=0 -> lower=-0.5 upper=0.5 effort=${effort} velocity=${velocity}
- joint gripper_right3_to_gripper_right1: limit lower=-0.5 upper=0.5 effort=1000 velocity=0 -> lower=-0.5 upper=0.5 effort=${effort} velocity=${velocity}
- joint joint2_to_joint1: limit lower=-3.14 upper=3.14159 effort=1000.0 velocity=0 -> lower=-3.14 upper=3.14159 effort=${effort} velocity=${velocity}
- joint joint3_to_joint2: limit lower=-3.14 upper=3.14159 effort=1000.0 velocity=0 -> lower=-3.14 upper=3.14159 effort=${effort} velocity=${velocity}
- joint joint4_to_joint3: limit lower=-3.14 upper=3.14159 effort=1000.0 velocity=0 -> lower=-3.14 upper=3.14159 effort=${effort} velocity=${velocity}
- joint joint5_to_joint4: limit lower=-3.14 upper=3.14159 effort=1000.0 velocity=0 -> lower=-3.14 upper=3.14159 effort=${effort} velocity=${velocity}
- joint joint6_to_joint5: limit lower=-3.14 upper=3.14159 effort=1000.0 velocity=0 -> lower=-3.14 upper=3.14159 effort=${effort} velocity=${velocity}
- joint joint6output_to_joint6: limit lower=-3.14 upper=3.14159 effort=1000.0 velocity=0 -> lower=-3.14 upper=3.14159 effort=${effort} velocity=${velocity}

Commit message: Added gripper to joint state

File: mycobot_280pi_description/urdf/mycobot_280_pi.urdf (robot description, URDF)
Before this commit: robot mycobot_280pi, 15 links, 14 joints
Joints:
- joint gripper_controller: limit lower=-0.8 upper=0.15 effort=${effort} velocity=${velocity} -> lower=-0.73 upper=0.15 effort=${effort} velocity=${velocity}

Commit message: Added gripper and its working

File: mycobot_280pi_description/urdf/mycobot_280_pi.urdf (robot description, URDF)
Before this commit: robot mycobot_280pi, 15 links, 14 joints
Joints:
- joint gripper_controller: limit lower=-0.73 upper=0.15 effort=${effort} velocity=${velocity} -> lower=-0.58 upper=0.15 effort=${effort} velocity=${velocity}

Commit message: Fixed gripper homing and working

File: mycobot_280pi_description/urdf/mycobot_280_pi.urdf (robot description, URDF)
Before this commit: robot mycobot_280pi, 15 links, 14 joints
Joints:
- joint joint6output_to_joint6: origin xyz=0 0.0456 0 rpy=-1.5708 0 0 -> xyz=0 0.0456 0 rpy=-1.5708 0.785398 0
